File: LS_weak.kicad_sch (KiCad schematic)
At the start: 7 parts, among them Q24 AO3400A

Commit message: Update LS_weak.kicad_sch
Parts:
- R16: LCSC C23162 -> (none)
Changed lines of the file:
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@@
 			)
 		)
-		(property "LCSC" "C23162"
+		(property "LCSC" ""
 			(at 125.73 96.52 0)
 			(effects
