File: VFRECU-VR.kicad_pcb (KiCad board)
At the start: 4 copper layers, 160 x 75.1 mm, 96 parts, among them IC2 LM1815MX_NOPB, IC2A1 LM1815MX_NOPB, J4 1-776087-1, J8 USB_B_Mini, M1 Module-power_12and5V-0.2, M2 Module-knock-0.2, M5 Module-wbo-0.5, M6 Module:mega-mcu100/0.2, M7 Module-wbo-0.5, Q1 ISL9V3040D3S, Q10 ZXMS6005SGTA, Q11 AO3400A, Q12 AO3400A, Q13 ZXMS6005SGTA, Q14 ZXMS6005SGTA, Q15 ZXMS6005SGTA, Q16 ZXMS6005SGTA, Q2 ISL9V3040D3S, Q3 ISL9V3040D3S, Q4 ISL9V3040D3S, Q7 ZXMS6005SGTA, Q8 ZXMS6005SGTA, Q9 ZXMS6005SGTA, U2 JDY-33

Commit message: Replace Vias
Parts:
- moved R24 9.50 mm to (242.0, 76.2)
- moved R32 2.61 mm to (241.7, 58.8)
Routing:
- net /IN_BUTTON3: track 191.8 -> 196.5 mm
- net /INJ4: track 163.9 -> 166.9 mm
- net /LS4: track 189.6 -> 187.0 mm
- net /OUT_LS2: track 80.7 -> 78.7 mm
- net /INJ3: track 199.9 -> 198.3 mm
- net /INJ1: track 167.4 -> 168.7 mm
- net /CAN+: track 215.9 -> 214.8 mm
- net /PWR_EN: track 75.6 -> 76.7 mm
- net /Clutch/kickstandswitch: track 75.8 -> 76.8 mm
- net /VIGN: track 68.6 -> 69.6 mm
- net /IGN1: track 60.6 -> 61.5 mm
- net /VR2: track 110.6 -> 109.8 mm
- net /CAN-: track 217.7 -> 218.5 mm
- net /INJ2: track 173.6 -> 174.3 mm
- net /LS1: track 200.3 -> 200.9 mm
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